Commit message: update wanfang's modification

File: ur_description/urdf/common.gazebo.xacro (robot description, xacro)
@@ -2,7 +2,7 @@
 <robot xmlns:xacro="http://ros.org/wiki/xacro">
   <gazebo>
-    <plugin name="ros_control" filename="libgazebo_ros_control.so">
-      <!--robotNamespace>/</robotNamespace-->
-      <!--robotSimType>gazebo_ros_control/DefaultRobotHWSim</robotSimType-->
+    <plugin name="gazebo_ros_control" filename="libgazebo_ros_control.so">
+      <robotNamespace>/ur5</robotNamespace>
+      <robotSimType>gazebo_ros_control/DefaultRobotHWSim</robotSimType>
     </plugin>
 <!--

File: ur_description/urdf/ur3_robot.urdf.xacro (robot description, xacro)
@@ -1,9 +1,13 @@
 <?xml version="1.0"?>
 <robot xmlns:xacro="http://ros.org/wiki/xacro"
-       name="ur3" >
+       name="ur3_kinect" >
   <!-- common stuff -->
   <xacro:include filename="$(find ur_description)/urdf/common.gazebo.xacro" />
   <!-- ur3 -->
   <xacro:include filename="$(find ur_description)/urdf/ur3.urdf.xacro" />
+  <!-- checkerboard -->
+  <xacro:include filename="$(find hector_components_description)/urdf/checkerboard.urdf.xacro" />
+  <!-- kinect camera -->
+  <xacro:include filename="$(find hector_sensors_description)/urdf/kinect_camera.urdf.xacro" />
   <!-- arm -->
   <xacro:ur3_robot prefix="" joint_limited="false"/>
@@ -14,3 +18,12 @@
     <origin xyz="0.0 0.0 0.0" rpy="0.0 0.0 0.0" />
   </joint>
+  <!-- end effector/checkbord -->
+  <xacro:checkerboard parent="ee_link" name="checkerboard" scaling="0.2">
+    <origin xyz="0.01 0.0 0.0" rpy="0.0 0.0 0.0"/>
+  </xacro:checkerboard>
+  <!-- kinect camare -->
+  <xacro:kinect_camera parent="base_link" name="kinect">
+    <!--origin xyz="0.2 0.1 1.0" rpy="0.0 ${pi/2} 0.0"/-->
+    <origin xyz="0.2 0.0 1.0" rpy="0.0 ${pi/2} 0.0"/>
+  </xacro:kinect_camera>
 </robot>

File: ur_description/urdf/ur5_joint_limited_robot.urdf.xacro (robot description, xacro)
@@ -2,8 +2,17 @@
 <robot xmlns:xacro="http://ros.org/wiki/xacro"
        name="ur5" >
+  <property name="prefix" value=""/>
+  <property name="M_PI" value="3.14159265359" />
   <!-- common stuff -->
   <xacro:include filename="$(find ur_description)/urdf/common.gazebo.xacro" />
   <!-- ur5 -->
   <xacro:include filename="$(find ur_description)/urdf/ur5.urdf.xacro" />
+  <!-- photoneo camera -->
+  <xacro:include filename="$(find phoxi_camera)/urdf/PhoXi3Dscanner_values.xacro"/> <!--Scanner values-->
+  <xacro:include filename="$(find phoxi_camera)/urdf/PhoXi3Dscanner_macro.xacro"/>  <!--Scanner macro-->
+  <!-- workplatform-->
+  <xacro:include filename="$(find ur_description)/urdf/platform.urdf.xacro" />
+  <!-- rg2 gripper -->
+  <xacro:include filename="$(find ur_description)/urdf/rg2.urdf.xacro" />
   <!-- arm -->
   <xacro:ur5_robot prefix="" joint_limited="true"
@@ -18,6 +27,18 @@
   <joint name="world_joint" type="fixed">
     <parent link="world" />
-    <child link = "base_link" />
+    <child link = "box" />
     <origin xyz="0.0 0.0 0.0" rpy="0.0 0.0 0.0" />
   </joint>
+  <!-- rg2 pipe -->
+  <!-- <xacro:rg2 prefix="${prefix}"/> -->
+  <!-- photoneo camare -->
+  <xacro:PhoXi3Dscanner scanner_parent = "base_link" scanner_name = "PhoXi3Dscanner" sensor_parent = "PhoXi3Dscanner" sensor_name = "PhoXi3Dscanner_sensor" >
+      <origin xyz="0.075 0.928 0.535" rpy="${pi-pi/6-pi/50} 0.02 0" /> <!--PhoXi3Dscanner origin-->
+      <xacro:PhoXi3DscannerS_default_sensor_origin /> <!--Extrinsic calibration data-->
+      <xacro:PhoXi3DscannerS_meshes /> <!--meshes-->
+  </xacro:PhoXi3Dscanner>
+  <!-- workplatform -->
+  <xacro:boxbase child="base_link" >
+    <origin xyz="0.0 0.0 ${boxz}" rpy="0.0 0.0 0.0"/>
+  </xacro:boxbase>
 </robot>

File: ur_description/urdf/ur5_robot.urdf.xacro (robot description, xacro)
@@ -2,15 +2,70 @@
 <robot xmlns:xacro="http://ros.org/wiki/xacro"
        name="ur5" >
+  <property name="prefix" value=""/>
+  <property name="M_PI" value="3.14159265359" />
   <!-- common stuff -->
   <xacro:include filename="$(find ur_description)/urdf/common.gazebo.xacro" />
   <!-- ur5 -->
   <xacro:include filename="$(find ur_description)/urdf/ur5.urdf.xacro" />
+  <!-- photoneo camera -->
+  <xacro:include filename="$(find phoxi_camera)/urdf/PhoXi3Dscanner_values.xacro"/> <!--Scanner values-->
+  <xacro:include filename="$(find phoxi_camera)/urdf/PhoXi3Dscanner_macro.xacro"/>  <!--Scanner macro-->
+  <!-- workplatform-->
+  <xacro:include filename="$(find ur_description)/urdf/platform.urdf.xacro" />
+  <!-- rg2 gripper -->
+  <xacro:include filename="$(find ur_description)/urdf/rg2.urdf.xacro" />
   <!-- arm -->
-  <xacro:ur5_robot prefix="" joint_limited="false"/>
+  <xacro:ur5_robot prefix="" joint_limited="true"
+    shoulder_pan_lower_limit="${-pi}" shoulder_pan_upper_limit="${pi}"
+    shoulder_lift_lower_limit="${-pi}" shoulder_lift_upper_limit="${pi}"
+    elbow_joint_lower_limit="${-pi}" elbow_joint_upper_limit="${pi}"
+    wrist_1_lower_limit="${-pi}" wrist_1_upper_limit="${pi}"
+    wrist_2_lower_limit="${-pi}" wrist_2_upper_limit="${pi}"
+    wrist_3_lower_limit="${-pi}" wrist_3_upper_limit="${pi}"
+  />
   <link name="world" />
   <joint name="world_joint" type="fixed">
     <parent link="world" />
-    <child link = "base_link" />
+    <child link = "box" />
     <origin xyz="0.0 0.0 0.0" rpy="0.0 0.0 0.0" />
   </joint>
+  <!-- gripper extender link -->
+  <joint name="gripper_extender_joint" type="fixed">
+    <origin rpy="0 0 0" xyz="0 0 0"/>
+    <parent link="${prefix}ee_link"/>
+    <child link="${prefix}gripper_extender_link"/>
+  </joint>
+  <link name="${prefix}gripper_extender_link">
+    <visual>
+      <geometry>
+        <cylinder length="0.218" radius="0.014"/>
+      </geometry>
+      <origin rpy="0 ${M_PI/2} 0" xyz="0.104 0.0 0.0"/>
+      <material name="White">
+        <color rgba="${150/255} ${150/255} ${150/255} 1.0"/>
+      </material>
+    </visual>
+    <collision>
+      <geometry>
+        <cylinder length="0.218" radius="0.014"/>
+      </geometry>
+      <origin rpy="0 ${M_PI/2} 0" xyz="0.104 0.0 0.00"/>
+    </collision>
+    <inertial>
+      <mass value="0.6"/>
+      <inertia ixx="1" ixy="0.0" ixz="0.0" iyy="1" iyz="0.0" izz="1"/>
+    </inertial>
+  </link>
+  <!-- rg2 pipe -->
+  <xacro:rg2 prefix="${prefix}"/>
+  <!-- photoneo camare -->
+  <xacro:PhoXi3Dscanner scanner_parent = "base_link" scanner_name = "PhoXi3Dscanner" sensor_parent = "PhoXi3Dscanner" sensor_name = "PhoXi3Dscanner_sensor" >
+      <origin xyz="0.085 0.915 0.535" rpy="${pi-pi/6-pi/50} 0.02 0" /> <!--PhoXi3Dscanner origin-->
+      <xacro:PhoXi3DscannerS_default_sensor_origin /> <!--Extrinsic calibration data-->
+      <xacro:PhoXi3DscannerS_meshes /> <!--meshes-->
+  </xacro:PhoXi3Dscanner>
+  <!-- workplatform -->
+  <xacro:boxbase child="base_link" >
+    <origin xyz="0.0 0.0 ${boxz}" rpy="0.0 0.0 0.0"/>
+  </xacro:boxbase>
 </robot>
