Commit message: 在ur5_robot.urdf.xacro中添加table，在ur5.urdf.xacro中将shoulder link到base（否则机器人坐标系会反向）

File: ur_description/urdf/ur5.urdf.xacro (robot description, xacro)
@@ -93,5 +93,5 @@
     </link>
     <joint name="${prefix}shoulder_pan_joint" type="revolute">
-      <parent link="${prefix}base_link" />
+      <parent link="${prefix}base" />
       <child link = "${prefix}shoulder_link" />
       <origin xyz="0.0 0.0 ${shoulder_height}" rpy="0.0 0.0 0.0" />

File: ur_description/urdf/ur5_robot.urdf.xacro (robot description, xacro)
@@ -8,4 +8,10 @@
   <!-- arm -->
   <xacro:ur5_robot prefix="" joint_limited="false"/>
+  <xacro:macro name="default_inertial" params="mass">
+    <inertial>
+      <mass value="${mass}" />
+      <inertia ixx="1.0" ixy="0.0" ixz="0.0" iyy="1.0" iyz="0.0" izz="1.0" />
+    </inertial>
+  </xacro:macro>
   <link name="world" />
   <joint name="world_joint" type="fixed">
@@ -14,3 +20,24 @@
     <origin xyz="0.0 0.0 0.0" rpy="0.0 0.0 0.0" />
   </joint>
+  <!-- table -->
+  <link name="tablebox">
+    <visual>
+      <geometry>
+        <box size="2 2.2 0.01"/>
+      </geometry>
+      <material name="gray"/>
+      <origin xyz="0 0 0.005" rpy="0 -0 0"/>
+    </visual>
+    <collision>
+      <geometry>
+        <box size="2 2.2 0.01"/>
+      </geometry>
+    </collision>
+    <xacro:default_inertial mass="1"/>
+  </link>
+  <joint name="world_table_joint" type="fixed">
+    <parent link="world" />
+    <child link = "tablebox" />
+    <origin xyz="0.0 -0.0 -0.00" rpy="0.0 0.0 0.0" />
+  </joint>
 </robot>
